Commit message: Updated link masses with values provided by Robotiq.

File: manipulation/models/robotiq_3f_description/urdf/robotiq-3f-gripper_articulated.urdf (robot description, URDF)
Before this commit: robot robotiq-3f-gripper_articulated, 13 links, 12 joints
Links:
- link finger_1_link_1: mass 0.15 -> 0.12622
- link finger_1_link_2: mass 0.15 -> 0.0601
- link finger_1_link_3: mass 0.05 -> 0.024
- link finger_2_link_1: mass 0.15 -> 0.12622
- link finger_2_link_2: mass 0.15 -> 0.0601
- link finger_2_link_3: mass 0.05 -> 0.024
- link finger_middle_link_1: mass 0.15 -> 0.12622
- link finger_middle_link_2: mass 0.15 -> 0.0601
- link finger_middle_link_3: mass 0.05 -> 0.024

Commit message: Updated mass of link_0 and link_1, added description of how Robotiq-provided mass values were used to calculate these values.

File: manipulation/models/robotiq_3f_description/urdf/robotiq-3f-gripper_articulated.urdf (robot description, URDF)
Before this commit: robot robotiq-3f-gripper_articulated, 13 links, 12 joints
Links:
- link finger_1_link_0: mass 0.05 -> 0.02133
- link finger_1_link_1: mass 0.12622 -> 0.10489
- link finger_2_link_0: mass 0.05 -> 0.02133
- link finger_2_link_1: mass 0.12622 -> 0.10489
- link finger_middle_link_0: mass 0.05 -> 0.02133
- link finger_middle_link_1: mass 0.12622 -> 0.10489
